File: Hardware/Ricardo-BlackBox/can.kicad_sch (KiCad schematic)
At the start: 11 parts, among them U2 SN65HVD230

Commit message: Initial hardware update
Parts:
- removed C18, C19: 220pF, Capacitor_SMD:C_0402_1005Metric, symbol Device:C_Small
- C17: value 0.1uF -> 47nF
- R10, R9: footprint Resistor_SMD:R_0402_1005Metric -> Resistor_SMD:R_0603_1608Metric
