File: Hardware/Ricardo-BlackBox/power.kicad_sch (KiCad schematic)
At the start: 21 parts, among them U3 LM66200DRLR, U4 MAX77827AEFD+T, U5 SC4215

Commit message: Initial hardware update
Parts:
- removed TP7: TestPoint, TestPoint:TestPoint_Pad_D1.5mm, symbol Connector:TestPoint
- U5: value SC4215 -> SC4215ASTRT; symbol iclr:RT9025-25GSP -> iclr:SC4215ASTRT
