File: Hardware/usb.kicad_sch (KiCad schematic)
At the start: 8 parts, among them J2 USB_C_Receptacle_USB2.0

Commit message: Updated footprints
Parts:
- J2: footprint Connector_USB:USB_C_Receptacle_Palconn_UTC16-G -> iclr:USB_C_Receptacle_Palconn_UTC16-G
- USBLED1: footprint Resistor_SMD:R_0402_1005Metric -> LED_SMD:LED_0402_1005Metric
Changed lines of the file:
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@@
 			)
 		)
-		(property "Footprint" "Connector_USB:USB_C_Receptacle_Palconn_UTC16-G"
+		(property "Footprint" "iclr:USB_C_Receptacle_Palconn_UTC16-G"
 			(at 104.14 104.14 0)
 			(effects
@@
 			)
 		)
-		(property "Footprint" "Resistor_SMD:R_0402_1005Metric"
+		(property "Footprint" "LED_SMD:LED_0402_1005Metric"
 			(at 162.56 92.71 90)
 			(effects

Commit message: Changed GPIO breakout to 8 pin connector
Changed lines of the file:
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@@
 (kicad_sch
-	(version 20231120)
+	(version 20250114)
 	(generator "eeschema")
-	(generator_version "8.0")
+	(generator_version "9.0")
 	(paper "A4")
 	(junction
